Commit message: fixed chapter 2

File: chapter_2_codes/mastering_ros_robot_description_pkg/urdf/diff_wheeled_robot.urdf (robot description, URDF)
Before this commit: robot differential_wheeled_robot, 7 links, 6 joints
Links:
- link base_link: mass 5 -> 5.0
Joints:
- joint caster_back_joint: origin xyz=-0.135 0.0 0.009 rpy=-1.57079632679 0 0 -> xyz=-0.135 0.0 0.009 rpy=-1.5707963 0 0
- joint caster_front_joint: origin xyz=0.115 0.0 0.007 rpy=-1.57079632679 0 0 -> xyz=0.115 0.0 0.007 rpy=-1.5707963 0 0
- joint front_left_wheel_joint: origin xyz=0.0 -0.15 0.0 rpy=0 0 0 -> xyz=0.0 0.15 0.0 rpy=0 0 0
- joint front_right_wheel_joint: origin xyz=0.0 0.15 0.0 rpy=0 0 0 -> xyz=0.0 -0.15 0.0 rpy=0 0 0

File: chapter_2_codes/mastering_ros_robot_description_pkg/urdf/diff_wheeled_robot.xacro (robot description, xacro)
@@ -1,6 +1,7 @@
 <?xml version="1.0"?>
-<robot name="differential_wheeled_robot" xmlns:xacro="http://www.ros.org/wiki/xacro">
+<robot name="differential_wheeled_robot"
+  xmlns:xacro="http://www.ros.org/wiki/xacro">
   <xacro:include filename="$(find mastering_ros_robot_description_pkg)/urdf/wheel.urdf.xacro" />
-<!-- Defining the colors used in this robot -->
+  <!-- Defining the colors used in this robot -->
   <material name="Black">
     <color rgba="0.0 0.0 0.0 1.0"/>
@@ -17,35 +18,37 @@
   <!-- PROPERTY LIST -->
   <!--All units in m-kg-s-radians unit system -->
-  <property name="M_PI" value="3.1415926535897931" />
-  <property name="M_PI_2" value="1.570796327" />
-  <property name="DEG_TO_RAD" value="0.017453293" />
+  <xacro:property name="M_PI" value="3.1415926535897931" />
+  <xacro:property name="M_PI_2" value="1.570796327" />
+  <xacro:property name="DEG_TO_RAD" value="0.017453293" />
   <!-- Main body radius and height -->
   <!-- Main Body Cylinder base   -->
-  <property name="base_height" value="0.02" />
-  <property name="base_radius" value="0.15" />
-  <property name="base_mass" value="5" /> <!-- in kg-->
+  <xacro:property name="base_height" value="0.02" />
+  <xacro:property name="base_radius" value="0.15" />
+  <xacro:property name="base_mass" value="5.0" />
+  <!-- in kg-->
   <!-- caster wheel radius and height -->
   <!-- caster wheel mass -->
-  <property name="caster_f_height" value="0.04" />
-  <property name="caster_f_radius" value="0.025" />
-  <property name="caster_f_mass" value="0.5" /> <!-- in kg-->
+  <xacro:property name="caster_f_height" value="0.04" />
+  <xacro:property name="caster_f_radius" value="0.025" />
+  <xacro:property name="caster_f_mass" value="0.5" />
+  <!-- in kg-->
   <!-- caster wheel radius and height -->
   <!-- caster wheel mass -->
-  <property name="caster_b_height" value="0.04" />
-  <property name="caster_b_radius" value="0.025" />
-  <property name="caster_b_mass" value="0.5" /> <!-- in kg-->
+  <xacro:property name="caster_b_height" value="0.04" />
+  <xacro:property name="caster_b_radius" value="0.025" />
+  <xacro:property name="caster_b_mass" value="0.5" />
+  <!-- in kg-->
   <!-- Wheels -->
-  <property name="wheel_mass" value="2.5" /> --> <!-- in kg-->
-  <property name="base_x_origin_to_wheel_origin" value="0.25" />
-  <property name="base_y_origin_to_wheel_origin" value="0.3" />
-  <property name="base_z_origin_to_wheel_origin" value="0.0" />
+  <xacro:property name="wheel_mass" value="2.5" />
+ -->  <!-- in kg-->
+  <xacro:property name="base_x_origin_to_wheel_origin" value="0.25" />
+  <xacro:property name="base_y_origin_to_wheel_origin" value="0.3" />
+  <xacro:property name="base_z_origin_to_wheel_origin" value="0.0" />
   <!-- Hokuyo Laser scanner -->
-  <property name="hokuyo_size" value="0.05" />
+  <xacro:property name="hokuyo_size" value="0.05" />
   <!-- Macro for calculating inertia of cylinder -->
-  <macro name="cylinder_inertia" params="m r h">
-    <inertia  ixx="${m*(3*r*r+h*h)/12}" ixy = "0" ixz = "0"
-              iyy="${m*(3*r*r+h*h)/12}" iyz = "0"
-              izz="${m*r*r/2}" />
-  </macro>
+  <xacro:macro name="cylinder_inertia" params="m r h">
+    <inertia ixx="${round(m*(3.0*r*r+h*h)/12.0,7)}" ixy = "0" ixz = "0" iyy="${round(m*(3.0*r*r+h*h)/12.0,7)}" iyz = "0" izz="${round(m*r*r/2.0,7)}" />
+  </xacro:macro>
   <!-- BASE-FOOTPRINT -->
   <!-- base_footprint is a fictitious link(frame) that is on the ground right below base_link origin -->
@@ -54,13 +57,11 @@
       <mass value="0.0001" />
       <origin xyz="0 0 0" />
-      <inertia ixx="0.0001" ixy="0.0" ixz="0.0"
-          iyy="0.0001" iyz="0.0"
-          izz="0.0001" />
-    </inertial>
-    <visual>
-        <origin xyz="0 0 0" rpy="0 0 0" />
-        <geometry>
-            <box size="0.001 0.001 0.001" />
-        </geometry>
+      <inertia ixx="0.0001" ixy="0.0" ixz="0.0" iyy="0.0001" iyz="0.0" izz="0.0001" />
+    </inertial>
+    <visual>
+      <origin xyz="0 0 0" rpy="0 0 0" />
+      <geometry>
+        <box size="0.001 0.001 0.001" />
+      </geometry>
     </visual>
   </link>
@@ -80,10 +81,10 @@
       <origin xyz="0 0 0" />
       <!--The 3x3 rotational inertia matrix. -->
-        <cylinder_inertia  m="${base_mass}" r="${base_radius}" h="${base_height}" />
+      <xacro:cylinder_inertia m="${base_mass}" r="${base_radius}" h="${base_height}" />
     </inertial>
     <visual>
       <origin xyz="0 0 0" rpy="0 0 0" />
       <geometry>
-          <cylinder length="${base_height}" radius="${base_radius}" />
+        <cylinder length="${base_height}" radius="${base_radius}" />
       </geometry>
       <material name="White" />
@@ -92,5 +93,5 @@
       <origin xyz="0 0 0" rpy="0 0 0 " />
       <geometry>
-          <cylinder length="${base_height}" radius="${base_radius}" />
+        <cylinder length="${base_height}" radius="${base_radius}" />
       </geometry>
     </collision>
@@ -100,69 +101,65 @@
     <turnGravityOff>false</turnGravityOff>
   </gazebo>
-<!--Caster front  -->
-    <link name="caster_front_link">
-    <visual>
-      <origin xyz="0 0.02 0" rpy="${M_PI/2} 0 0" />
-      <geometry>
-	<sphere radius="${caster_f_radius}" />
+  <!--Caster front  -->
+  <link name="caster_front_link">
+    <visual>
+      <origin xyz="0 0.02 0" rpy="${round(M_PI/2.0,7)} 0 0" />
+      <geometry>
+        <sphere radius="${caster_f_radius}" />
       </geometry>
       <material name="Black" />
     </visual>
-      <collision>
-        <geometry>
-	<sphere radius="${caster_f_radius}" />
-        </geometry>
-      <origin xyz="0 0.02 0" rpy="${M_PI/2} 0 0" />
-      </collision>
-      <inertial>
-        <mass value="${caster_f_mass}" />
-        <origin xyz="0 0 0" />
-        <inertia ixx="0.001" ixy="0.0" ixz="0.0"
-                 iyy="0.001" iyz="0.0"
-                 izz="0.001" />
-      </inertial>
-    </link>
- <joint name="caster_front_joint" type="fixed">
-      <parent link="base_link"/>
-      <child link="caster_front_link"/>
-      <origin xyz="0.115 0.0 0.007" rpy="${-M_PI/2} 0 0"/>
-    </joint>
+    <collision>
+      <geometry>
+        <sphere radius="${caster_f_radius}" />
+      </geometry>
+      <origin xyz="0 0.02 0" rpy="${round(M_PI/2.0,7)} 0 0" />
+    </collision>
+    <inertial>
+      <mass value="${caster_f_mass}" />
+      <origin xyz="0 0 0" />
+      <inertia ixx="0.001" ixy="0.0" ixz="0.0" iyy="0.001" iyz="0.0" izz="0.001" />
+    </inertial>
+  </link>
+  <joint name="caster_front_joint" type="fixed">
+    <parent link="base_link"/>
+    <child link="caster_front_link"/>
+    <origin xyz="0.115 0.0 0.007" rpy="${round(-M_PI/2.0,7)} 0 0"/>
+  </joint>
   <gazebo reference="caster_front_link">
     <turnGravityOff>false</turnGravityOff>
   </gazebo>
-<!--Caster back  -->
-    <link name="caster_back_link">
-    <visual>
-      <origin xyz="0.02 0.02 0 " rpy="${M_PI/2} 0 0" />
-      <geometry>
-	<sphere radius="${caster_b_radius}" />
+  <!--Caster back  -->
+  <link name="caster_back_link">
+    <visual>
+      <origin xyz="0.02 0.02 0 " rpy="${round(M_PI/2.0,7)} 0 0" />
+      <geometry>
+        <sphere radius="${caster_b_radius}" />
       </geometry>
       <material name="Black" />
     </visual>
-      <collision>
-        <geometry>
-		<sphere radius="${caster_b_radius}" />
-        </geometry>
-      <origin xyz="0 0.02 0 " rpy="${M_PI/2} 0 0" />
-      </collision>
-      <inertial>
-        <mass value="${caster_b_mass}" />
-        <origin xyz="0 0 0" />
-        <inertia ixx="0.001" ixy="0.0" ixz="0.0"
-                 iyy="0.001" iyz="0.0"
-                 izz="0.001" />
-      </inertial>
-    </link>
-    <joint name="caster_back_joint" type="fixed">
-      <parent link="base_link"/>
-      <child link="caster_back_link"/>
-      <origin xyz="-0.135 0.0 0.009" rpy="${-M_PI/2} 0 0"/>
-    </joint>
+    <collision>
+      <geometry>
+        <sphere radius="${caster_b_radius}" />
+      </geometry>
+      <origin xyz="0 0.02 0 " rpy="${round(M_PI/2.0,7)} 0 0" />
+    </collision>
+    <inertial>
+      <mass value="${caster_b_mass}" />
+      <origin xyz="0 0 0" />
+      <inertia ixx="0.001" ixy="0.0" ixz="0.0" iyy="0.001" iyz="0.0" izz="0.001" />
+    </inertial>
+  </link>
+  <joint name="caster_back_joint" type="fixed">
+    <parent link="base_link"/>
+    <child link="caster_back_link"/>
+    <origin xyz="-0.135 0.0 0.009" rpy="${round(-M_PI/2.0,7)} 0 0"/>
+  </joint>
   <gazebo reference="caster_back_link">
     <turnGravityOff>false</turnGravityOff>
   </gazebo>
-<!-- Wheel Definitions -->
-  <wheel fb="front" lr="right" parent="base_link" translateX="0" translateY="0.5" flipY="1"/>
-  <wheel fb="front" lr="left" parent="base_link" translateX="0" translateY="-0.5" flipY="1"/>
+  <!-- Wheel Definitions -->
+  <xacro:wheel fb="front" lr="right" parent="base_link" translateX="0" translateY="-0.5" flipY="1.0"/>
+  <xacro:wheel fb="front" lr="left" parent="base_link" translateX="0" translateY="0.5" flipY="1.0"/>
   <!-- SENSORS -->
   <!-- hokuyo -->
@@ -177,5 +174,5 @@
   </link>
   <joint name="hokuyo_joint" type="fixed">
-    <origin xyz="${base_radius - hokuyo_size/2} 0 ${base_height+hokuyo_size/4}" rpy="0 0 0" />
+    <origin xyz="${base_radius - hokuyo_size/2.0} 0 ${base_height+hokuyo_size/4.0}" rpy="0 0 0" />
     <parent link="base_link"/>
     <child link="hokuyo_link" />
@@ -185,5 +182,5 @@
     <turnGravityOff>false</turnGravityOff>
     <sensor type="ray" name="head_hokuyo_sensor">
-      <pose>${hokuyo_size/2} 0 0 0 0 0</pose>
+      <pose>${hokuyo_size/2.0} 0 0 0 0 0</pose>
       <visualize>false</visualize>
       <update_rate>40</update_rate>

File: chapter_2_codes/mastering_ros_robot_description_pkg/urdf/pan_tilt.urdf (robot description, URDF)
Before this commit: robot pan_tilt, 3 links, 2 joints
Links:
- link tilt_link: geometry collision cylinder length=0.4 radius=0.24000000000000002; visual cylinder length=0.4 radius=0.04

File: chapter_2_codes/mastering_ros_robot_description_pkg/urdf/pan_tilt.xacro (robot description, xacro)
@@ -1,26 +1,23 @@
 <?xml version="1.0"?>
 <robot xmlns:xacro="http://www.ros.org/wiki/xacro"
- 	xmlns:sensor="http://playerstage.sourceforge.net/gazebo/xmlschema/#sensor"
-    	xmlns:controller="http://playerstage.sourceforge.net/gazebo/xmlschema/#controller"
-    	xmlns:interface="http://playerstage.sourceforge.net/gazebo/xmlschema/#interface"
-	name="pan_tilt">
-	<xacro:property name="base_link_length" value="0.01" />
-	<xacro:property name="base_link_radius" value="0.2" />
-	<xacro:property name="pan_link_length" value="0.4" />
-	<xacro:property name="pan_link_radius" value="0.04" />
-	<xacro:property name="tilt_link_length" value="0.4" />
-	<xacro:property name="tilt_link_radius" value="0.04" />
-	<xacro:macro name="inertial_matrix" params="mass">
-               <inertial>
-                       <mass value="${mass}" />
-                       <inertia ixx="0.5" ixy="0.0" ixz="0.0"
-                                iyy="0.5" iyz="0.0"
-                                izz="0.5" />
-               </inertial>
-	</xacro:macro>
+  xmlns:sensor="http://playerstage.sourceforge.net/gazebo/xmlschema/#sensor"
+  xmlns:controller="http://playerstage.sourceforge.net/gazebo/xmlschema/#controller"
+  xmlns:interface="http://playerstage.sourceforge.net/gazebo/xmlschema/#interface" name="pan_tilt">
+  <xacro:property name="base_link_length" value="0.01" />
+  <xacro:property name="base_link_radius" value="0.2" />
+  <xacro:property name="pan_link_length" value="0.4" />
+  <xacro:property name="pan_link_radius" value="0.04" />
+  <xacro:property name="tilt_link_length" value="0.4" />
+  <xacro:property name="tilt_link_radius" value="0.04" />
+  <xacro:macro name="inertial_matrix" params="mass">
+    <inertial>
+      <mass value="${mass}" />
+      <inertia ixx="0.5" ixy="0.0" ixz="0.0" iyy="0.5" iyz="0.0" izz="0.5" />
+    </inertial>
+  </xacro:macro>
   <link name="base_link">
     <visual>
       <geometry>
-	<cylinder length="${base_link_length}" radius="${base_link_radius}"/>
+        <cylinder length="${base_link_length}" radius="${base_link_radius}"/>
       </geometry>
       <origin rpy="0 0 0" xyz="0 0 0"/>
@@ -31,9 +28,9 @@
     <collision>
       <geometry>
-	<cylinder length="${base_link_length+0.02}" radius="0.2"/>
+        <cylinder length="${base_link_length+0.02}" radius="0.2"/>
       </geometry>
       <origin rpy="0 0 0" xyz="0 0 0"/>
     </collision>
-	<xacro:inertial_matrix mass="1"/>
+    <xacro:inertial_matrix mass="1"/>
   </link>
   <joint name="pan_joint" type="revolute">
@@ -48,5 +45,5 @@
     <visual>
       <geometry>
-	<cylinder length="${pan_link_length}" radius="${pan_link_radius}"/>
+        <cylinder length="${pan_link_length}" radius="${pan_link_radius}"/>
       </geometry>
       <origin rpy="0 0 0" xyz="0 0 0.09"/>
@@ -57,9 +54,9 @@
     <collision>
       <geometry>
-	<cylinder length="${pan_link_length}" radius="${pan_link_radius+0.02}"/>
+        <cylinder length="${pan_link_length}" radius="${pan_link_radius+0.02}"/>
       </geometry>
       <origin rpy="0 0 0" xyz="0 0 0.09"/>
     </collision>
-	<xacro:inertial_matrix mass="1"/>
+    <xacro:inertial_matrix mass="1"/>
   </link>
   <joint name="tilt_joint" type="revolute">
@@ -74,5 +71,5 @@
     <visual>
       <geometry>
-	<cylinder length="${tilt_link_length}" radius="${tilt_link_radius}"/>
+        <cylinder length="${tilt_link_length}" radius="${tilt_link_radius}"/>
       </geometry>
       <origin rpy="0 1.5 0" xyz="0 0 0"/>
@@ -83,9 +80,9 @@
     <collision>
       <geometry>
-	<cylinder length="${tilt_link_length}" radius="${tilt_link_radius+0.2}"/>
+        <cylinder length="${tilt_link_length}" radius="${tilt_link_radius+0.2}"/>
       </geometry>
       <origin rpy="0 1.5 0" xyz="0 0 0"/>
     </collision>
-	<xacro:inertial_matrix mass="1"/>
+    <xacro:inertial_matrix mass="1"/>
   </link>
 </robot>

File: chapter_2_codes/mastering_ros_robot_description_pkg/urdf/seven_dof_arm.urdf (robot description, URDF)
Before this commit: robot seven_dof_arm, 18 links, 17 joints
Links:
- link rgbd_camera_depth_frame: mass 0.001 -> None
- link rgbd_camera_depth_optical_frame: mass 0.001 -> None
- link rgbd_camera_optical_frame: mass 0.001 -> None
- link rgbd_camera_rgb_frame: mass 0.001 -> None
- link rgbd_camera_rgb_optical_frame: mass 0.001 -> None
Joints:
- joint finger_joint1: limit lower=0 upper=0.03 effort=100 velocity=1.0 -> lower=0 upper=0.03 effort=1 velocity=1.0
- joint gripper_roll_joint: origin xyz=0 0 0.080 rpy=4.712385 -1.570795 0 -> xyz=0 0 0.080 rpy=4.712384999999999 -1.570795 0
- joint rgbd_camera_depth_optical_joint: origin xyz=0 0 0 rpy=-1.57079632679 0.0 -1.57079632679 -> xyz=0 0 0 rpy=-1.5707963267948966 0.0 -1.5707963267948966
- joint rgbd_camera_joint: origin xyz=0.1 0 1 rpy=0 1.308996939 0 -> (none)
- joint rgbd_camera_optical_joint: origin xyz=0 0 0 rpy=-1.57079632679 0 -1.57079632679 -> (none)
- joint rgbd_camera_rgb_optical_joint: origin xyz=0 0 0 rpy=-1.57079632679 0.0 -1.57079632679 -> xyz=0 0 0 rpy=-1.5707963267948966 0.0 -1.5707963267948966

File: chapter_2_codes/mastering_ros_robot_description_pkg/urdf/seven_dof_arm.xacro (robot description, xacro)
@@ -11,44 +11,44 @@
         <color rgba="1.0 1.0 1.0 1.0"/>
     </material>
-  <property name="deg_to_rad" value="0.01745329251994329577"/>
+  <xacro:property name="deg_to_rad" value="0.01745329251994329577"/>
   <!-- Constants -->
-  <property name="M_SCALE" value="0.001 0.001 0.001"/>
-  <property name="M_PI" value="3.14159"/>
+  <xacro:property name="M_SCALE" value="0.001 0.001 0.001"/>
+  <xacro:property name="M_PI" value="3.14159"/>
   <!-- Shoulder pan link properties -->
-  <property name="shoulder_pan_width" value="0.04" />
-  <property name="shoulder_pan_len" value="0.08" />
+  <xacro:property name="shoulder_pan_width" value="0.04" />
+  <xacro:property name="shoulder_pan_len" value="0.08" />
   <!-- Shoulder pitch link properties -->
-  <property name="shoulder_pitch_len" value="0.14" />
-  <property name="shoulder_pitch_width" value="0.04" />
-  <property name="shoulder_pitch_height" value="0.04" />
+  <xacro:property name="shoulder_pitch_len" value="0.14" />
+  <xacro:property name="shoulder_pitch_width" value="0.04" />
+  <xacro:property name="shoulder_pitch_height" value="0.04" />
   <!-- Elbow roll link properties -->
-  <property name="elbow_roll_width" value="0.02" />
-  <property name="elbow_roll_len" value="0.06" />
+  <xacro:property name="elbow_roll_width" value="0.02" />
+  <xacro:property name="elbow_roll_len" value="0.06" />
   <!-- Elbow pitch link properties -->
-  <property name="elbow_pitch_len" value="0.22" />
-  <property name="elbow_pitch_width" value="0.04" />
-  <property name="elbow_pitch_height" value="0.04" />
+  <xacro:property name="elbow_pitch_len" value="0.22" />
+  <xacro:property name="elbow_pitch_width" value="0.04" />
+  <xacro:property name="elbow_pitch_height" value="0.04" />
   <!-- Wrist roll link properties -->
-  <property name="wrist_roll_width" value="0.02" />
-  <property name="wrist_roll_len" value="0.04" />
+  <xacro:property name="wrist_roll_width" value="0.02" />
+  <xacro:property name="wrist_roll_len" value="0.04" />
   <!-- wrist pitch link properties -->
-  <property name="wrist_pitch_len" value="0.06" />
-  <property name="wrist_pitch_width" value="0.04" />
-  <property name="wrist_pitch_height" value="0.04" />
+  <xacro:property name="wrist_pitch_len" value="0.06" />
+  <xacro:property name="wrist_pitch_width" value="0.04" />
+  <xacro:property name="wrist_pitch_height" value="0.04" />
   <!-- Gripper roll link properties -->
-  <property name="gripper_roll_width" value="0.04" />
-  <property name="gripper_roll_len" value="0.02" />
+  <xacro:property name="gripper_roll_width" value="0.04" />
+  <xacro:property name="gripper_roll_len" value="0.02" />
   <!-- Left gripper -->
-  <property name="left_gripper_len" value="0.08" />
-  <property name="left_gripper_width" value="0.01" />
-  <property name="left_gripper_height" value="0.01" />
+  <xacro:property name="left_gripper_len" value="0.08" />
+  <xacro:property name="left_gripper_width" value="0.01" />
+  <xacro:property name="left_gripper_height" value="0.01" />
   <!-- Right gripper -->
-  <property name="right_gripper_len" value="0.08" />
-  <property name="right_gripper_width" value="0.01" />
-  <property name="right_gripper_height" value="0.01" />
+  <xacro:property name="right_gripper_len" value="0.08" />
+  <xacro:property name="right_gripper_width" value="0.01" />
+  <xacro:property name="right_gripper_height" value="0.01" />
   <!-- Right gripper -->
-  <property name="grasp_frame_len" value="0.02" />
-  <property name="grasp_frame_width" value="0.02" />
-  <property name="grasp_frame_height" value="0.02" />
+  <xacro:property name="grasp_frame_len" value="0.02" />
+  <xacro:property name="grasp_frame_width" value="0.02" />
+  <xacro:property name="grasp_frame_height" value="0.02" />
    <xacro:macro name="inertial_matrix" params="mass">
       <inertial>
@@ -324,9 +324,11 @@
     <origin xyz="0.0 0 0" />
     <axis xyz="0 1 0" />
-      <limit effort="100" lower="0" upper="0.03" velocity="1.0"/>
+      <limit effort="1" lower="0" upper="0.03" velocity="1.0"/>
+	<!--
       <safety_controller k_position="20"
                          k_velocity="20"
                          soft_lower_limit="${-0.15 }"
                          soft_upper_limit="${ 0.0 }"/>
+	-->
     <dynamics damping="50" friction="1"/>
   </joint>
@@ -404,8 +406,9 @@
    <xacro:transmission_block joint_name="finger_joint1"/>
    <xacro:transmission_block joint_name="finger_joint2"/>
-  <!-- Define arm with gripper mounted on a base -->
+  <!-- Define arm with gripper mounted on a base
   <xacro:base name="base"/>
   <xacro:arm parent="base"/>
   <xacro:gripper parent="tool"/>
+		-->
   <!-- Define RGB-D sensor -->
   <xacro:xtion_pro_live name="rgbd_camera" parent="base">
