Commit message: fixed chapter 2

File: chapter_2_codes/mastering_ros_robot_description_pkg/urdf/wheel.urdf.xacro (robot description, xacro)
@@ -1,20 +1,20 @@
 <?xml version="1.0"?>
-<robot name="wheel" xmlns:xacro="http://www.ros.org/wiki/xacro">
+<robot name="wheel"
+  xmlns:xacro="http://www.ros.org/wiki/xacro">
   <!-- Wheels -->
-  <property name="wheel_radius" value="0.04" />
-  <property name="wheel_height" value="0.02" />
-  <property name="wheel_mass" value="2.5" /> <!-- in kg-->
-  <property name="base_x_origin_to_wheel_origin" value="0.25" />
-  <property name="base_y_origin_to_wheel_origin" value="0.3" />
-  <property name="base_z_origin_to_wheel_origin" value="0.0" />
-  <macro name="cylinder_inertia" params="m r h">
-    <inertia  ixx="${m*(3*r*r+h*h)/12}" ixy = "0" ixz = "0"
-              iyy="${m*(3*r*r+h*h)/12}" iyz = "0"
-              izz="${m*r*r/2}" />
-  </macro>
-  <xacro:macro name="wheel" params="fb lr parent translateX translateY flipY"> <!--fb : front, back ; lr: left, right -->
+  <xacro:property name="wheel_radius" value="0.04" />
+  <xacro:property name="wheel_height" value="0.02" />
+  <xacro:property name="wheel_mass" value="2.5" />
+  <!-- in kg-->
+  <xacro:property name="base_x_origin_to_wheel_origin" value="0.25" />
+  <xacro:property name="base_y_origin_to_wheel_origin" value="0.3" />
+  <xacro:property name="base_z_origin_to_wheel_origin" value="0.0" />
+  <xacro:macro name="cylinder_inertia" params="m r h">
+    <inertia ixx="${round(m*(3.0*r*r+h*h)/12.0,7)}" ixy = "0.0" ixz = "0.0" iyy="${round(m*(3.0*r*r+h*h)/12.0,7)}" iyz = "0.0" izz="${round(m*r*r/2.0,7)}" />
+  </xacro:macro>
+  <xacro:macro name="wheel" params="fb lr parent translateX translateY flipY">    <!--fb : front, back ; lr: left, right -->
     <link name="${fb}_${lr}_wheel">
       <visual>
-        <origin xyz="0 0 0" rpy="${flipY*M_PI/2} 0  0 " />
+        <origin xyz="0 0 0" rpy="${round(flipY*M_PI/2.0,7)} 0  0 " />
         <geometry>
           <cylinder length="${wheel_height}" radius="${wheel_radius}" />
@@ -23,5 +23,5 @@
       </visual>
       <collision>
-        <origin xyz="0 0 0" rpy="${flipY*M_PI/2} 0 0 " />
+        <origin xyz="0 0 0" rpy="${round(flipY*M_PI/2.0,7)} 0 0 " />
         <geometry>
           <cylinder length="${wheel_height}" radius="${wheel_radius}" />
@@ -31,5 +31,5 @@
         <mass value="${wheel_mass}" />
         <origin xyz="0 0 0" />
-        <cylinder_inertia  m="${wheel_mass}" r="${wheel_radius}" h="${wheel_height}" />
+        <xacro:cylinder_inertia m="${wheel_mass}" r="${wheel_radius}" h="${wheel_height}" />
       </inertial>
     </link>
@@ -37,6 +37,6 @@
       <mu1 value="1.0"/>
       <mu2 value="1.0"/>
-      <kp  value="10000000.0" />
-      <kd  value="1.0" />
+      <kp value="10000000.0" />
+      <kd value="1.0" />
       <fdir1 value="1 0 0"/>
       <material>Gazebo/Grey</material>
@@ -46,5 +46,5 @@
       <parent link="${parent}"/>
       <child link="${fb}_${lr}_wheel"/>
-      <origin xyz="${translateX * base_x_origin_to_wheel_origin} ${translateY * base_y_origin_to_wheel_origin} ${base_z_origin_to_wheel_origin}" rpy="0 0 0" />
+      <origin xyz="${round(translateX * base_x_origin_to_wheel_origin,7)} ${round(translateY * base_y_origin_to_wheel_origin,7)} ${base_z_origin_to_wheel_origin}" rpy="0 0 0" />
       <axis xyz="0 1 0" rpy="0  0" />
       <limit effort="100" velocity="100"/>
